Commit message: updated urdf and code to match lab4

File: urdf/fingeredu.urdf (robot description, URDF)
Before this commit: robot fingeredu, 6 links, 5 joints
Joints:
- joint finger_base_to_upper_joint: axis -1 0 0 -> 1 0 0
- joint finger_middle_to_lower_joint: axis 0 1 0 -> 0 -1 0
- joint finger_upper_to_middle_joint: axis 0 1 0 -> 0 -1 0
